File: Spartanpods_v2 (SquarePCB)/Spartanpods_v2 (Square).kicad_pcb (KiCad board)
At the start: 2 copper layers, 100 x 105 mm, 24 parts, among them Q2 Q_Photo_NPN, Q3 BC847, SW1 SW_DP3T

Commit message: Included Library Package
Parts:
- BT1: footprint !MyFootprints:CR2032-Holder -> Spartanpods_FootprintLibrary:CR2032-Holder
- D1, D2, D3, D4, D5: footprint !MyFootprints:LED - MyPLCC2 (RoundMask_LED Side) -> Spartanpods_FootprintLibrary:LED - MyPLCC2 (RoundMask_LED Side)
- FID1, FID2, FID3, FID4: footprint Fiducial:Fiducial_0.75mm_Mask2.25mm -> Spartanpods_FootprintLibrary:Fiducial_0.75mm_Mask2.25mm
- G1: footprint !MyFootprints:JD3_Diode -> Spartanpods_FootprintLibrary:JD3_Diode
- G2: footprint Spartanpods:Combined -> Spartanpods_FootprintLibrary:Combined
- Pot1: footprint Potentiometer_SMD:Potentiometer_Bourns_TC33X_Vertical -> Spartanpods_FootprintLibrary:Potentiometer_Bourns_TC33X_Vertical
- Q2: footprint !MyFootprints:PhotoTrans_PT12-21C_TR8 (Flipped) -> Spartanpods_FootprintLibrary:PhotoTrans_PT12-21C_TR8 (Flipped)
- Q3: footprint Package_TO_SOT_SMD:SOT-23 -> Spartanpods_FootprintLibrary:SOT-23
- R1: footprint Capacitor_SMD:C_0603_1608Metric_Pad1.08x0.95mm_HandSolder -> Spartanpods_FootprintLibrary:C_0603_1608Metric_Pad1.08x0.95mm_HandSolder
- R2, R3, R4, R5, R6: footprint Capacitor_SMD:C_0805_2012Metric_Pad1.18x1.45mm_HandSolder -> Spartanpods_FootprintLibrary:C_0805_2012Metric_Pad1.18x1.45mm_HandSolder
- REF**: footprint Spartanpods:Untitled -> Spartanpods_FootprintLibrary:Untitled
- REF**: footprint Spartanpods:MiniLogo -> Spartanpods_FootprintLibrary:MiniLogo
- SW1: footprint !MyFootprints:DP3T - JS203011SCQN -> Spartanpods_FootprintLibrary:DP3T - JS203011SCQN
Changed lines of the file:
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@@
 	(net 16 "unconnected-(SW1-Pad5)")
 	(net 17 "unconnected-(SW1-Pad2)")
-	(footprint "Spartanpods:Combined"
+	(footprint "Spartanpods_FootprintLibrary:Combined"
 		(locked yes)
 		(layer "F.Cu")
@@
 		(embedded_fonts no)
 	)
-	(footprint "Capacitor_SMD:C_0805_2012Metric_Pad1.18x1.45mm_HandSolder"
+	(footprint "Spartanpods_FootprintLibrary:C_0805_2012Metric_Pad1.18x1.45mm_HandSolder"
 		(layer "B.Cu")
 		(at 155.956 56.3665 90)
@@
 		)
 	)
-	(footprint "Capacitor_SMD:C_0805_2012Metric_Pad1.18x1.45mm_HandSolder"
+	(footprint "Spartanpods_FootprintLibrary:C_0805_2012Metric_Pad1.18x1.45mm_HandSolder"
 		(layer "B.Cu")
 		(at 139.9032 86.614 180)
@@
 		)
 	)
-	(footprint "Fiducial:Fiducial_0.75mm_Mask2.25mm"
+	(footprint "Spartanpods_FootprintLibrary:Fiducial_0.75mm_Mask2.25mm"
 		(layer "B.Cu")
 		(at 197.953609 34.349936)
@@
 		(embedded_fonts no)
 	)
-	(footprint "Potentiometer_SMD:Potentiometer_Bourns_TC33X_Vertical"
+	(footprint "Spartanpods_FootprintLibrary:Potentiometer_Bourns_TC33X_Vertical"
 		(layer "B.Cu")
 		(at 174.852 110.0836)
@@
 		)
 	)
-	(footprint "Spartanpods:Untitled"
+	(footprint "Spartanpods_FootprintLibrary:Untitled"
 		(layer "B.Cu")
 		(at 169.7736 85.09 180)
@@
 		(embedded_fonts no)
 	)
-	(footprint "!MyFootprints:DP3T - JS203011SCQN"
+	(footprint "Spartanpods_FootprintLibrary:DP3T - JS203011SCQN"
 		(layer "B.Cu")
 		(at 142.9644 127.2923 -90)
@@
 		)
 	)
-	(footprint "Fiducial:Fiducial_0.75mm_Mask2.25mm"
+	(footprint "Spartanpods_FootprintLibrary:Fiducial_0.75mm_Mask2.25mm"
 		(layer "B.Cu")
 		(at 100.953609 136.349936)
@@
 		(embedded_fonts no)
 	)
-	(footprint "!MyFootprints:PhotoTrans_PT12-21C_TR8 (Flipped)"
+	(footprint "Spartanpods_FootprintLibrary:PhotoTrans_PT12-21C_TR8 (Flipped)"
 		(layer "B.Cu")
 		(at 197.4088 87.2668 90)
@@
 		)
 	)
-	(footprint "Fiducial:Fiducial_0.75mm_Mask2.25mm"
+	(footprint "Spartanpods_FootprintLibrary:Fiducial_0.75mm_Mask2.25mm"
 		(layer "B.Cu")
 		(at 197.953609 136.349936)
@@
 		(embedded_fonts no)
 	)
-	(footprint "Capacitor_SMD:C_0805_2012Metric_Pad1.18x1.45mm_HandSolder"
+	(footprint "Spartanpods_FootprintLibrary:C_0805_2012Metric_Pad1.18x1.45mm_HandSolder"
 		(layer "B.Cu")
 		(at 174.5996 77.8764)
@@
 		)
 	)
-	(footprint "Spartanpods:MiniLogo"
+	(footprint "Spartanpods_FootprintLibrary:MiniLogo"
 		(layer "B.Cu")
 		(at 128.4732 63.754 180)
@@
 		(embedded_fonts no)
 	)
-	(footprint "Capacitor_SMD:C_0805_2012Metric_Pad1.18x1.45mm_HandSolder"
+	(footprint "Spartanpods_FootprintLibrary:C_0805_2012Metric_Pad1.18x1.45mm_HandSolder"
 		(layer "B.Cu")
 		(at 170.5864 71.8312)
@@
 		)
 	)
-	(footprint "!MyFootprints:CR2032-Holder"
+	(footprint "Spartanpods_FootprintLibrary:CR2032-Holder"
 		(layer "B.Cu")
 		(at 130.0988 106.6292 180)
@@
 		)
 	)
-	(footprint "Capacitor_SMD:C_0805_2012Metric_Pad1.18x1.45mm_HandSolder"
+	(footprint "Spartanpods_FootprintLibrary:C_0805_2012Metric_Pad1.18x1.45mm_HandSolder"
 		(layer "B.Cu")
 		(at 149.0472 54.61 90)
@@
 		)
 	)
-	(footprint "!MyFootprints:LED - MyPLCC2 (RoundMask_LED Side)"
+	(footprint "Spartanpods_FootprintLibrary:LED - MyPLCC2 (RoundMask_LED Side)"
 		(layer "B.Cu")
 		(at 172.466 59.1312 -145)
@@
 		)
 	)
-	(footprint "!MyFootprints:LED - MyPLCC2 (RoundMask_LED Side)"
+	(footprint "Spartanpods_FootprintLibrary:LED - MyPLCC2 (RoundMask_LED Side)"
 		(layer "B.Cu")
 		(at 178.8252 72.0852 180)
@@
 		)
 	)
-	(footprint "Package_TO_SOT_SMD:SOT-23"
+	(footprint "Spartanpods_FootprintLibrary:SOT-23"
 		(layer "B.Cu")
 		(at 194.2744 107.5713 180)
@@
 		)
 	)
-	(footprint "!MyFootprints:LED - MyPLCC2 (RoundMask_LED Side)"
+	(footprint "Spartanpods_FootprintLibrary:LED - MyPLCC2 (RoundMask_LED Side)"
 		(layer "B.Cu")
 		(at 162.578099 49.432204 -125)
@@
 		)
 	)
-	(footprint "!MyFootprints:LED - MyPLCC2 (RoundMask_LED Side)"
+	(footprint "Spartanpods_FootprintLibrary:LED - MyPLCC2 (RoundMask_LED Side)"
 		(layer "B.Cu")
 		(at 149.9616 46.168 -90)
@@
 		)
 	)
-	(footprint "!MyFootprints:LED - MyPLCC2 (RoundMask_LED Side)"
+	(footprint "Spartanpods_FootprintLibrary:LED - MyPLCC2 (RoundMask_LED Side)"
 		(layer "B.Cu")
 		(at 130.2512 86.4108)
@@
 		)
 	)
-	(footprint "Fiducial:Fiducial_0.75mm_Mask2.25mm"
+	(footprint "Spartanpods_FootprintLibrary:Fiducial_0.75mm_Mask2.25mm"
 		(layer "B.Cu")
 		(at 100.953609 34.349936)
@@
 		(embedded_fonts no)
 	)
-	(footprint "!MyFootprints:JD3_Diode"
+	(footprint "Spartanpods_FootprintLibrary:JD3_Diode"
 		(layer "B.Cu")
 		(at 108.2548 128.1684 180)
@@
 		(embedded_fonts no)
 	)
-	(footprint "Capacitor_SMD:C_0603_1608Metric_Pad1.08x0.95mm_HandSolder"
+	(footprint "Spartanpods_FootprintLibrary:C_0603_1608Metric_Pad1.08x0.95mm_HandSolder"
 		(layer "B.Cu")
 		(at 162.7124 108.8644 180)
@@
 		(effects
 			(font
-				(size 0.64 0.64)
+				(size 0.8 0.8)
 				(thickness 0.15)
 			)
@@
 		(effects
 			(font
-				(size 0.64 0.64)
+				(size 0.8 0.8)
 				(thickness 0.15)
 			)
@@
 	)
 	(gr_text "Phototransistor"
-		(at 195.58 85.7504 0)
+		(at 194.7164 85.7504 0)
 		(layer "B.SilkS")
 		(effects
 			(font
-				(size 0.64 0.64)
+				(size 0.8 0.8)
 				(thickness 0.15)
 			)
