File: Spartanpods_v2 (SquarePCB)/Spartanpods_v2 (Square).kicad_sch (KiCad schematic)
At the start: 22 parts, among them Q2 Phototransistor, Q3 BC847, SW1 SW_DP3T

Commit message: Included Library Package
Parts:
- BT1: symbol !MyLibrary:Battery_Cell -> Spartanpods_SymbolLibrary:Battery_Cell
- D1, D2, D3, D4, D5: symbol Device:LED -> Spartanpods_SymbolLibrary:LED
- FID1, FID2, FID3, FID4: symbol Mechanical:Fiducial -> Spartanpods_SymbolLibrary:Fiducial
- G1: symbol !MyLibrary:JD3_Diode -> Spartanpods_SymbolLibrary:JD3_Diode
- G2: symbol Graphic:Logo_Open_Hardware_Small -> Spartanpods_SymbolLibrary:Logo_Open_Hardware_Small
- Pot1: symbol Device:R_Potentiometer_US -> Spartanpods_SymbolLibrary:R_Potentiometer_US
- Q2: symbol !MyLibrary:Q_Photo_NPN -> Spartanpods_SymbolLibrary:Q_Photo_NPN
- Q3: symbol Transistor_BJT:BC847 -> Spartanpods_SymbolLibrary:BC847
- R1, R2, R3, R4, R5, R6: symbol Device:R_US -> Spartanpods_SymbolLibrary:R_US
- SW1: symbol Switch:SW_DP3T -> Spartanpods_SymbolLibrary:SW_DP3T
Changed lines of the file:
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@@
 	)
 	(symbol
-		(lib_id "Mechanical:Fiducial")
+		(lib_id "Spartanpods_SymbolLibrary:Fiducial")
 		(at 267.97 140.97 0)
 		(unit 1)
@@
 	)
 	(symbol
-		(lib_id "power:PWR_FLAG")
+		(lib_id "Spartanpods_SymbolLibrary:PWR_FLAG")
 		(at 76.2 81.28 90)
 		(unit 1)
@@
 	)
 	(symbol
-		(lib_id "Device:LED")
+		(lib_id "Spartanpods_SymbolLibrary:LED")
 		(at 194.31 80.01 90)
 		(unit 1)
@@
 	)
 	(symbol
-		(lib_id "Device:R_US")
+		(lib_id "Spartanpods_SymbolLibrary:R_US")
 		(at 194.31 71.12 0)
 		(unit 1)
@@
 	)
 	(symbol
-		(lib_id "Device:R_US")
+		(lib_id "Spartanpods_SymbolLibrary:R_US")
 		(at 156.21 71.12 0)
 		(unit 1)
@@
 	)
 	(symbol
-		(lib_id "power:+3.3V")
+		(lib_id "Spartanpods_SymbolLibrary:+3.3V")
 		(at 76.2 66.04 0)
 		(unit 1)
@@
 	)
 	(symbol
-		(lib_id "Device:LED")
+		(lib_id "Spartanpods_SymbolLibrary:LED")
 		(at 181.61 80.01 90)
 		(unit 1)
@@
 	)
 	(symbol
-		(lib_id "Graphic:Logo_Open_Hardware_Small")
+		(lib_id "Spartanpods_SymbolLibrary:Logo_Open_Hardware_Small")
 		(at 226.06 157.48 0)
 		(unit 1)
@@
 	)
 	(symbol
-		(lib_id "Switch:SW_DP3T")
+		(lib_id "Spartanpods_SymbolLibrary:SW_DP3T")
 		(at 92.71 121.92 0)
 		(unit 1)
@@
 	)
 	(symbol
-		(lib_id "Device:R_US")
+		(lib_id "Spartanpods_SymbolLibrary:R_US")
 		(at 170.18 71.12 0)
 		(unit 1)
@@
 	)
 	(symbol
-		(lib_id "Device:LED")
+		(lib_id "Spartanpods_SymbolLibrary:LED")
 		(at 170.18 80.01 90)
 		(unit 1)
@@
 	)
 	(symbol
-		(lib_id "Device:LED")
+		(lib_id "Spartanpods_SymbolLibrary:LED")
 		(at 156.21 80.01 90)
 		(unit 1)
@@
 	)
 	(symbol
-		(lib_id "Device:R_Potentiometer_US")
+		(lib_id "Spartanpods_SymbolLibrary:R_Potentiometer_US")
 		(at 116.84 90.17 0)
 		(unit 1)
@@
 	)
 	(symbol
-		(lib_id "Mechanical:Fiducial")
+		(lib_id "Spartanpods_SymbolLibrary:Fiducial")
 		(at 267.97 153.67 0)
 		(unit 1)
@@
 	)
 	(symbol
-		(lib_id "Mechanical:Fiducial")
+		(lib_id "Spartanpods_SymbolLibrary:Fiducial")
 		(at 267.97 160.02 0)
 		(unit 1)
@@
 	)
 	(symbol
-		(lib_id "power:GNDREF")
+		(lib_id "Spartanpods_SymbolLibrary:GNDREF")
 		(at 76.2 125.73 0)
 		(unit 1)
@@
 	)
 	(symbol
-		(lib_id "Transistor_BJT:BC847")
+		(lib_id "Spartanpods_SymbolLibrary:BC847")
 		(at 142.24 100.33 0)
 		(unit 1)
@@
 	)
 	(symbol
-		(lib_id "Device:LED")
+		(lib_id "Spartanpods_SymbolLibrary:LED")
 		(at 207.01 80.01 90)
 		(unit 1)
@@
 	)
 	(symbol
-		(lib_id "Mechanical:Fiducial")
+		(lib_id "Spartanpods_SymbolLibrary:Fiducial")
 		(at 267.97 147.32 0)
 		(unit 1)
@@
 	)
 	(symbol
-		(lib_id "Device:R_US")
+		(lib_id "Spartanpods_SymbolLibrary:R_US")
 		(at 207.01 71.12 0)
 		(unit 1)
@@
 	)
 	(symbol
-		(lib_id "Device:R_US")
+		(lib_id "Spartanpods_SymbolLibrary:R_US")
 		(at 181.61 71.12 0)
 		(unit 1)
@@
 	)
 	(symbol
-		(lib_id "Device:R_US")
+		(lib_id "Spartanpods_SymbolLibrary:R_US")
 		(at 116.84 76.2 0)
 		(mirror x)
@@
 	)
 	(symbol
-		(lib_id "Switch:SW_DP3T")
+		(lib_id "Spartanpods_SymbolLibrary:SW_DP3T")
 		(at 92.71 133.35 0)
 		(unit 2)
@@
 	)
 	(symbol
-		(lib_id "!MyLibrary:Battery_Cell")
+		(lib_id "Spartanpods_SymbolLibrary:Battery_Cell")
 		(at 76.2 95.25 0)
 		(mirror y)
@@
 	)
 	(symbol
-		(lib_id "!MyLibrary:JD3_Diode")
+		(lib_id "Spartanpods_SymbolLibrary:JD3_Diode")
 		(at 241.3 157.48 0)
 		(unit 1)
@@
 	)
 	(symbol
-		(lib_id "!MyLibrary:Q_Photo_NPN")
+		(lib_id "Spartanpods_SymbolLibrary:Q_Photo_NPN")
 		(at 121.92 107.95 0)
 		(unit 1)
@@
 	)
 	(symbol
-		(lib_id "power:PWR_FLAG")
+		(lib_id "Spartanpods_SymbolLibrary:PWR_FLAG")
 		(at 76.2 106.68 90)
 		(unit 1)
