File: Spartanpods_v1 (Independent Text Wave)/Spartanpods.kicad_sch (KiCad schematic)
At the start: 20 parts, among them Q2 Q_Photo_NPN, Q3 BC847, SW1 SW_SPDT

Commit message: Full Library Update
Parts:
- BT1: symbol !MyLibrary:Battery_Cell -> Spartanpods_WaveTextSymbolsLibrary:Battery_Cell
- D1, D2, D3, D4: symbol Device:LED -> Spartanpods_WaveTextSymbolsLibrary:LED
- FID1, FID2, FID3, FID4: symbol Mechanical:Fiducial -> Spartanpods_WaveTextSymbolsLibrary:Fiducial
- G1: symbol !MyLibrary:JD3_Diode -> Spartanpods_WaveTextSymbolsLibrary:JD3_Diode
- G2: symbol Graphic:Logo_Open_Hardware_Small -> Spartanpods_WaveTextSymbolsLibrary:Logo_Open_Hardware_Small
- Pot1: symbol Device:R_Potentiometer_US -> Spartanpods_WaveTextSymbolsLibrary:R_Potentiometer_US
- Q2: symbol !MyLibrary:Q_Photo_NPN -> Spartanpods_WaveTextSymbolsLibrary:Q_Photo_NPN
- Q3: symbol Transistor_BJT:BC847 -> Spartanpods_WaveTextSymbolsLibrary:BC847
- R1, R2, R3, R4, R5: symbol Device:R_US -> Spartanpods_WaveTextSymbolsLibrary:R_US
- SW1: symbol Switch:SW_SPDT -> Spartanpods_WaveTextSymbolsLibrary:SW_SPDT
Changed lines of the file:
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@@
 	)
 	(symbol
-		(lib_id "Mechanical:Fiducial")
+		(lib_id "Spartanpods_WaveTextSymbolsLibrary:Fiducial")
 		(at 267.97 140.97 0)
 		(unit 1)
@@
 	)
 	(symbol
-		(lib_id "power:PWR_FLAG")
+		(lib_id "Spartanpods_WaveTextSymbolsLibrary:PWR_FLAG")
 		(at 76.2 81.28 90)
 		(unit 1)
@@
 	)
 	(symbol
-		(lib_id "Device:LED")
+		(lib_id "Spartanpods_WaveTextSymbolsLibrary:LED")
 		(at 194.31 80.01 90)
 		(unit 1)
@@
 	)
 	(symbol
-		(lib_id "Device:R_US")
+		(lib_id "Spartanpods_WaveTextSymbolsLibrary:R_US")
 		(at 194.31 71.12 0)
 		(unit 1)
@@
 	)
 	(symbol
-		(lib_id "Device:R_US")
+		(lib_id "Spartanpods_WaveTextSymbolsLibrary:R_US")
 		(at 156.21 71.12 0)
 		(unit 1)
@@
 	)
 	(symbol
-		(lib_id "power:+3.3V")
+		(lib_id "Spartanpods_WaveTextSymbolsLibrary:+3.3V")
 		(at 76.2 66.04 0)
 		(unit 1)
@@
 	)
 	(symbol
-		(lib_id "Device:LED")
+		(lib_id "Spartanpods_WaveTextSymbolsLibrary:LED")
 		(at 181.61 80.01 90)
 		(unit 1)
@@
 	)
 	(symbol
-		(lib_id "Graphic:Logo_Open_Hardware_Small")
+		(lib_id "Spartanpods_WaveTextSymbolsLibrary:Logo_Open_Hardware_Small")
 		(at 226.06 157.48 0)
 		(unit 1)
-		(exclude_from_sim no)
+		(exclude_from_sim yes)
 		(in_bom yes)
 		(on_board yes)
@@
 			)
 		)
-		(property "Sim.Enable" "0"
-			(at 226.06 157.48 0)
-			(effects
-				(font
-					(size 1.27 1.27)
-				)
-				(hide yes)
-			)
-		)
 		(instances
 			(project ""
@@
 	)
 	(symbol
-		(lib_id "Device:R_US")
+		(lib_id "Spartanpods_WaveTextSymbolsLibrary:R_US")
 		(at 170.18 71.12 0)
 		(unit 1)
@@
 	)
 	(symbol
-		(lib_id "Device:LED")
+		(lib_id "Spartanpods_WaveTextSymbolsLibrary:LED")
 		(at 170.18 80.01 90)
 		(unit 1)
@@
 	)
 	(symbol
-		(lib_id "Device:LED")
+		(lib_id "Spartanpods_WaveTextSymbolsLibrary:LED")
 		(at 156.21 80.01 90)
 		(unit 1)
@@
 	)
 	(symbol
-		(lib_id "Device:R_Potentiometer_US")
+		(lib_id "Spartanpods_WaveTextSymbolsLibrary:R_Potentiometer_US")
 		(at 116.84 90.17 0)
 		(unit 1)
@@
 	)
 	(symbol
-		(lib_id "Mechanical:Fiducial")
+		(lib_id "Spartanpods_WaveTextSymbolsLibrary:Fiducial")
 		(at 267.97 153.67 0)
 		(unit 1)
@@
 	)
 	(symbol
-		(lib_id "Mechanical:Fiducial")
+		(lib_id "Spartanpods_WaveTextSymbolsLibrary:Fiducial")
 		(at 267.97 160.02 0)
 		(unit 1)
@@
 	)
 	(symbol
-		(lib_id "power:GNDREF")
+		(lib_id "Spartanpods_WaveTextSymbolsLibrary:GNDREF")
 		(at 76.2 125.73 0)
 		(unit 1)
@@
 	)
 	(symbol
-		(lib_id "Transistor_BJT:BC847")
+		(lib_id "Spartanpods_WaveTextSymbolsLibrary:BC847")
 		(at 142.24 100.33 0)
 		(unit 1)
@@
 	)
 	(symbol
-		(lib_id "Switch:SW_SPDT")
+		(lib_id "Spartanpods_WaveTextSymbolsLibrary:SW_SPDT")
 		(at 92.71 121.92 0)
 		(unit 1)
@@
 	)
 	(symbol
-		(lib_id "Mechanical:Fiducial")
+		(lib_id "Spartanpods_WaveTextSymbolsLibrary:Fiducial")
 		(at 267.97 147.32 0)
 		(unit 1)
@@
 	)
 	(symbol
-		(lib_id "Device:R_US")
+		(lib_id "Spartanpods_WaveTextSymbolsLibrary:R_US")
 		(at 181.61 71.12 0)
 		(unit 1)
@@
 	)
 	(symbol
-		(lib_id "Device:R_US")
+		(lib_id "Spartanpods_WaveTextSymbolsLibrary:R_US")
 		(at 116.84 76.2 0)
 		(mirror x)
@@
 	)
 	(symbol
-		(lib_id "!MyLibrary:Battery_Cell")
+		(lib_id "Spartanpods_WaveTextSymbolsLibrary:Battery_Cell")
 		(at 76.2 95.25 0)
 		(mirror y)
@@
 	)
 	(symbol
-		(lib_id "!MyLibrary:JD3_Diode")
+		(lib_id "Spartanpods_WaveTextSymbolsLibrary:JD3_Diode")
 		(at 241.3 157.48 0)
 		(unit 1)
@@
 	)
 	(symbol
-		(lib_id "!MyLibrary:Q_Photo_NPN")
+		(lib_id "Spartanpods_WaveTextSymbolsLibrary:Q_Photo_NPN")
 		(at 121.92 107.95 0)
 		(unit 1)
@@
 	)
 	(symbol
-		(lib_id "power:PWR_FLAG")
+		(lib_id "Spartanpods_WaveTextSymbolsLibrary:PWR_FLAG")
 		(at 76.2 106.68 90)
 		(unit 1)
