File: Spartanpods_v4 (Square +LED Letters)/Spartanpods_v4 (Square +LED Letters).kicad_pcb (KiCad board)
At the start: 2 copper layers, 100 x 105 mm, 35 parts, among them Q2 Phototransistor, Q3 BC847, SW1 SW_DP3T

Commit message: Tidy
Parts:
- BT1: footprint !MyFootprints:CR2032-Holder -> SpartanpodsV4_FootprintLibrary:CR2032-Holder
- D1, D10, D2, D3, D4, D5, D6, D7, D8, D9: footprint !MyFootprints:LED - MyPLCC2 (RoundMask_LED Side) -> SpartanpodsV4_FootprintLibrary:LED - MyPLCC2 (RoundMask_LED Side)
- FID1, FID2, FID3, FID4: footprint Fiducial:Fiducial_0.75mm_Mask2.25mm -> SpartanpodsV4_FootprintLibrary:Fiducial_0.75mm_Mask2.25mm
- G1: footprint !MyFootprints:JD3_Diode -> SpartanpodsV4_FootprintLibrary:JD3_Diode
- G2: footprint Spartanpods:Combined_LED Text -> SpartanpodsV4_FootprintLibrary:Combined_LED Text
- Pot1: footprint Potentiometer_SMD:Potentiometer_Bourns_TC33X_Vertical -> SpartanpodsV4_FootprintLibrary:Potentiometer_Bourns_TC33X_Vertical
- Q2: footprint !MyFootprints:PhotoTrans_PT12-21C_TR8 (Flipped) -> SpartanpodsV4_FootprintLibrary:PhotoTrans_PT12-21C_TR8 (Flipped)
- Q3: footprint Package_TO_SOT_SMD:SOT-23 -> SpartanpodsV4_FootprintLibrary:SOT-23
- R1: footprint Capacitor_SMD:C_0603_1608Metric_Pad1.08x0.95mm_HandSolder -> SpartanpodsV4_FootprintLibrary:C_0603_1608Metric_Pad1.08x0.95mm_HandSolder
- R10, R11, R2, R3, R4, R5, R6, R7, R8, R9: footprint Capacitor_SMD:C_0805_2012Metric_Pad1.18x1.45mm_HandSolder -> SpartanpodsV4_FootprintLibrary:C_0805_2012Metric_Pad1.18x1.45mm_HandSolder
- R12: footprint Resistor_SMD:R_0805_2012Metric_Pad1.20x1.40mm_HandSolder -> SpartanpodsV4_FootprintLibrary:R_0805_2012Metric_Pad1.20x1.40mm_HandSolder
- REF**: footprint Spartanpods_FootprintLibrary:Untitled -> SpartanpodsV4_FootprintLibrary:Untitled
- REF**: footprint Spartanpods_FootprintLibrary:MiniLogo -> SpartanpodsV4_FootprintLibrary:MiniLogo
- SW1: footprint !MyFootprints:DP3T - JS203011SCQN -> SpartanpodsV4_FootprintLibrary:DP3T - JS203011SCQN
Changed lines of the file:
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@@
 	(net 22 "unconnected-(SW1-Pad4)")
 	(net 23 "Net-(R10-Pad1)")
-	(footprint "Spartanpods:Combined_LED Text"
+	(footprint "SpartanpodsV4_FootprintLibrary:Combined_LED Text"
 		(layer "F.Cu")
 		(at 99.453609 137.849936)
@@
 		(embedded_fonts no)
 	)
-	(footprint "Capacitor_SMD:C_0805_2012Metric_Pad1.18x1.45mm_HandSolder"
+	(footprint "SpartanpodsV4_FootprintLibrary:C_0805_2012Metric_Pad1.18x1.45mm_HandSolder"
 		(layer "B.Cu")
 		(at 155.956 56.3665 90)
@@
 		)
 	)
-	(footprint "Capacitor_SMD:C_0805_2012Metric_Pad1.18x1.45mm_HandSolder"
+	(footprint "SpartanpodsV4_FootprintLibrary:C_0805_2012Metric_Pad1.18x1.45mm_HandSolder"
 		(layer "B.Cu")
 		(at 139.9032 86.614 180)
@@
 		)
 	)
-	(footprint "Fiducial:Fiducial_0.75mm_Mask2.25mm"
+	(footprint "SpartanpodsV4_FootprintLibrary:Fiducial_0.75mm_Mask2.25mm"
 		(layer "B.Cu")
 		(at 197.953609 34.349936)
@@
 		(embedded_fonts no)
 	)
-	(footprint "Potentiometer_SMD:Potentiometer_Bourns_TC33X_Vertical"
+	(footprint "SpartanpodsV4_FootprintLibrary:Potentiometer_Bourns_TC33X_Vertical"
 		(layer "B.Cu")
 		(at 181.2068 90.8132)
@@
 		)
 	)
-	(footprint "Spartanpods_FootprintLibrary:Untitled"
+	(footprint "SpartanpodsV4_FootprintLibrary:Untitled"
 		(layer "B.Cu")
 		(at 169.7736 85.09 180)
@@
 		(embedded_fonts no)
 	)
-	(footprint "!MyFootprints:DP3T - JS203011SCQN"
+	(footprint "SpartanpodsV4_FootprintLibrary:DP3T - JS203011SCQN"
 		(layer "B.Cu")
 		(at 152.5524 103.6828 -90)
@@
 		)
 	)
-	(footprint "Fiducial:Fiducial_0.75mm_Mask2.25mm"
+	(footprint "SpartanpodsV4_FootprintLibrary:Fiducial_0.75mm_Mask2.25mm"
 		(layer "B.Cu")
 		(at 100.953609 136.349936)
@@
 		(embedded_fonts no)
 	)
-	(footprint "Capacitor_SMD:C_0805_2012Metric_Pad1.18x1.45mm_HandSolder"
+	(footprint "SpartanpodsV4_FootprintLibrary:C_0805_2012Metric_Pad1.18x1.45mm_HandSolder"
 		(layer "B.Cu")
 		(at 132.0292 119.6848 -90)
@@
 		)
 	)
-	(footprint "!MyFootprints:PhotoTrans_PT12-21C_TR8 (Flipped)"
+	(footprint "SpartanpodsV4_FootprintLibrary:PhotoTrans_PT12-21C_TR8 (Flipped)"
 		(layer "B.Cu")
 		(at 197.4596 43.6372 90)
@@
 		)
 	)
-	(footprint "Fiducial:Fiducial_0.75mm_Mask2.25mm"
+	(footprint "SpartanpodsV4_FootprintLibrary:Fiducial_0.75mm_Mask2.25mm"
 		(layer "B.Cu")
 		(at 197.953609 136.349936)
@@
 		(embedded_fonts no)
 	)
-	(footprint "!MyFootprints:LED - MyPLCC2 (RoundMask_LED Side)"
+	(footprint "SpartanpodsV4_FootprintLibrary:LED - MyPLCC2 (RoundMask_LED Side)"
 		(layer "B.Cu")
 		(at 183.5912 128.4224 90)
@@
 		)
 	)
-	(footprint "Capacitor_SMD:C_0805_2012Metric_Pad1.18x1.45mm_HandSolder"
+	(footprint "SpartanpodsV4_FootprintLibrary:C_0805_2012Metric_Pad1.18x1.45mm_HandSolder"
 		(layer "B.Cu")
 		(at 174.5996 77.8764)
@@
 		)
 	)
-	(footprint "Spartanpods_FootprintLibrary:MiniLogo"
+	(footprint "SpartanpodsV4_FootprintLibrary:MiniLogo"
 		(layer "B.Cu")
 		(at 128.4732 63.754 180)
@@
 		(embedded_fonts no)
 	)
-	(footprint "Capacitor_SMD:C_0805_2012Metric_Pad1.18x1.45mm_HandSolder"
+	(footprint "SpartanpodsV4_FootprintLibrary:C_0805_2012Metric_Pad1.18x1.45mm_HandSolder"
 		(layer "B.Cu")
 		(at 147.828 119.7864 -90)
@@
 		)
 	)
-	(footprint "!MyFootprints:LED - MyPLCC2 (RoundMask_LED Side)"
+	(footprint "SpartanpodsV4_FootprintLibrary:LED - MyPLCC2 (RoundMask_LED Side)"
 		(layer "B.Cu")
 		(at 115.9256 128.4224 90)
@@
 		)
 	)
-	(footprint "Capacitor_SMD:C_0805_2012Metric_Pad1.18x1.45mm_HandSolder"
+	(footprint "SpartanpodsV4_FootprintLibrary:C_0805_2012Metric_Pad1.18x1.45mm_HandSolder"
 		(layer "B.Cu")
 		(at 170.5864 71.8312)
@@
 		)
 	)
-	(footprint "Capacitor_SMD:C_0805_2012Metric_Pad1.18x1.45mm_HandSolder"
+	(footprint "SpartanpodsV4_FootprintLibrary:C_0805_2012Metric_Pad1.18x1.45mm_HandSolder"
 		(layer "B.Cu")
 		(at 112.4712 119.6633 -90)
@@
 		)
 	)
-	(footprint "!MyFootprints:CR2032-Holder"
+	(footprint "SpartanpodsV4_FootprintLibrary:CR2032-Holder"
 		(layer "B.Cu")
 		(at 120.5484 101.0412 180)
@@
 		)
 	)
-	(footprint "Capacitor_SMD:C_0805_2012Metric_Pad1.18x1.45mm_HandSolder"
+	(footprint "SpartanpodsV4_FootprintLibrary:C_0805_2012Metric_Pad1.18x1.45mm_HandSolder"
 		(layer "B.Cu")
 		(at 149.0472 54.61 90)
@@
 		)
 	)
-	(footprint "!MyFootprints:LED - MyPLCC2 (RoundMask_LED Side)"
+	(footprint "SpartanpodsV4_FootprintLibrary:LED - MyPLCC2 (RoundMask_LED Side)"
 		(layer "B.Cu")
 		(at 172.466 59.1312 -145)
@@
 		)
 	)
-	(footprint "!MyFootprints:LED - MyPLCC2 (RoundMask_LED Side)"
+	(footprint "SpartanpodsV4_FootprintLibrary:LED - MyPLCC2 (RoundMask_LED Side)"
 		(layer "B.Cu")
 		(at 178.8252 72.0852 180)
@@
 		)
 	)
-	(footprint "Package_TO_SOT_SMD:SOT-23"
+	(footprint "SpartanpodsV4_FootprintLibrary:SOT-23"
 		(layer "B.Cu")
 		(at 194.3608 58.8123 180)
@@
 		)
 	)
-	(footprint "!MyFootprints:LED - MyPLCC2 (RoundMask_LED Side)"
+	(footprint "SpartanpodsV4_FootprintLibrary:LED - MyPLCC2 (RoundMask_LED Side)"
 		(layer "B.Cu")
 		(at 162.578099 49.432204 -125)
@@
 		)
 	)
-	(footprint "Resistor_SMD:R_0805_2012Metric_Pad1.20x1.40mm_HandSolder"
+	(footprint "SpartanpodsV4_FootprintLibrary:R_0805_2012Metric_Pad1.20x1.40mm_HandSolder"
 		(layer "B.Cu")
 		(at 142.24 112.0648 -90)
@@
 		)
 	)
-	(footprint "!MyFootprints:LED - MyPLCC2 (RoundMask_LED Side)"
+	(footprint "SpartanpodsV4_FootprintLibrary:LED - MyPLCC2 (RoundMask_LED Side)"
 		(layer "B.Cu")
 		(at 149.9616 46.168 -90)
@@
 		)
 	)
-	(footprint "!MyFootprints:LED - MyPLCC2 (RoundMask_LED Side)"
+	(footprint "SpartanpodsV4_FootprintLibrary:LED - MyPLCC2 (RoundMask_LED Side)"
 		(layer "B.Cu")
 		(at 130.2512 86.4108)
@@
 		)
 	)
-	(footprint "Fiducial:Fiducial_0.75mm_Mask2.25mm"
+	(footprint "SpartanpodsV4_FootprintLibrary:Fiducial_0.75mm_Mask2.25mm"
 		(layer "B.Cu")
 		(at 100.953609 34.349936)
@@
 		(embedded_fonts no)
 	)
-	(footprint "!MyFootprints:LED - MyPLCC2 (RoundMask_LED Side)"
+	(footprint "SpartanpodsV4_FootprintLibrary:LED - MyPLCC2 (RoundMask_LED Side)"
 		(layer "B.Cu")
 		(at 148.0509 128.3208 90)
@@
 		)
 	)
-	(footprint "!MyFootprints:LED - MyPLCC2 (RoundMask_LED Side)"
+	(footprint "SpartanpodsV4_FootprintLibrary:LED - MyPLCC2 (RoundMask_LED Side)"
 		(layer "B.Cu")
 		(at 166.0341 128.3208 90)
@@
 		)
 	)
-	(footprint "!MyFootprints:JD3_Diode"
+	(footprint "SpartanpodsV4_FootprintLibrary:JD3_Diode"
 		(layer "B.Cu")
 		(at 105.5664 128.4224 180)
@@
 		(embedded_fonts no)
 	)
-	(footprint "Capacitor_SMD:C_0805_2012Metric_Pad1.18x1.45mm_HandSolder"
+	(footprint "SpartanpodsV4_FootprintLibrary:C_0805_2012Metric_Pad1.18x1.45mm_HandSolder"
 		(layer "B.Cu")
 		(at 183.5912 119.9388 -90)
@@
 		)
 	)
-	(footprint "Capacitor_SMD:C_0805_2012Metric_Pad1.18x1.45mm_HandSolder"
+	(footprint "SpartanpodsV4_FootprintLibrary:C_0805_2012Metric_Pad1.18x1.45mm_HandSolder"
 		(layer "B.Cu")
 		(at 166.0144 119.9388 -90)
@@
 		)
 	)
-	(footprint "Capacitor_SMD:C_0603_1608Metric_Pad1.08x0.95mm_HandSolder"
+	(footprint "SpartanpodsV4_FootprintLibrary:C_0603_1608Metric_Pad1.08x0.95mm_HandSolder"
 		(layer "B.Cu")
 		(at 170.7896 90.7796 180)
@@
 		)
 	)
-	(footprint "!MyFootprints:LED - MyPLCC2 (RoundMask_LED Side)"
+	(footprint "SpartanpodsV4_FootprintLibrary:LED - MyPLCC2 (RoundMask_LED Side)"
 		(layer "B.Cu")
 		(at 132.2832 128.3208 90)
