File: Spartanpods_v4 (Square +LED Letters)/Spartanpods_v4 (Square +LED Letters).kicad_sch (KiCad schematic)
At the start: 33 parts, among them Q2 Phototransistor, Q3 BC847, SW1 SW_DP3T

Commit message: Tidy
Parts:
- BT1: symbol Spartanpods_SymbolLibrary:Battery_Cell -> Spartanpods_v4_SymbolLibrary:Battery_Cell
- D1, D10, D2, D3, D4, D5, D6, D7, D8, D9: symbol Spartanpods_SymbolLibrary:LED -> Spartanpods_v4_SymbolLibrary:LED
- FID1, FID2, FID3, FID4: symbol Spartanpods_SymbolLibrary:Fiducial -> Spartanpods_v4_SymbolLibrary:Fiducial
- G1: symbol Spartanpods_SymbolLibrary:JD3_Diode -> Spartanpods_v4_SymbolLibrary:JD3_Diode
- G2: footprint Spartanpods:Combined -> Spartanpods:Combined_LED Text; symbol Spartanpods_SymbolLibrary:Logo_Open_Hardware_Small -> Spartanpods_v4_SymbolLibrary:Logo_Open_Hardware_Small
- Pot1: symbol Spartanpods_SymbolLibrary:R_Potentiometer_US -> Spartanpods_v4_SymbolLibrary:R_Potentiometer_US
- Q2: symbol Spartanpods_SymbolLibrary:Q_Photo_NPN -> Spartanpods_v4_SymbolLibrary:Q_Photo_NPN
- Q3: symbol Spartanpods_SymbolLibrary:BC847 -> Spartanpods_v4_SymbolLibrary:BC847
- R1, R10, R11, R2, R3, R4, R5, R6, R7, R8, R9: symbol Spartanpods_SymbolLibrary:R_US -> Spartanpods_v4_SymbolLibrary:R_US
- R12: footprint (none) -> Resistor_SMD:R_0805_2012Metric_Pad1.20x1.40mm_HandSolder; symbol Device:R_US -> Spartanpods_v4_SymbolLibrary:R_US
- SW1: footprint (none) -> !MyFootprints:DP3T - JS203011SCQN; symbol Spartanpods_SymbolLibrary:SW_DP3T -> Spartanpods_v4_SymbolLibrary:SW_DP3T
Connections:
- net +3.3V: now also R12.1; no longer R10.1, R11.1, R7.1, R8.1, R9.1
- net at D1.1 (K), D10.1 (K), D2.1 (K)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: no longer R12.1, R12.2
- new net: R10.1, R11.1, R12.2, R7.1, R8.1, R9.1
Other:
- moved on the sheet: R12
Changed lines of the file:
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@@
 	)
 	(junction
-		(at 163.83 86.36)
-		(diameter 0)
-		(color 0 0 0 0)
-	)
-	(junction
 		(at 124.46 100.33)
 		(diameter 0)
@@
 	)
 	(junction
-		(at 163.83 93.98)
-		(diameter 0)
-		(color 0 0 0 0)
-	)
-	(junction
 		(at 179.07 66.04)
 		(diameter 0)
@@
 	(wire
 		(pts
-			(xy 156.21 86.36) (xy 163.83 86.36)
+			(xy 156.21 86.36) (xy 179.07 86.36)
 		)
 		(stroke
@@
 	(wire
 		(pts
+			(xy 223.52 66.04) (xy 227.33 66.04)
+		)
+		(stroke
+			(width 0)
+			(type default)
+		)
+	)
+	(wire
+		(pts
 			(xy 257.81 67.31) (xy 257.81 66.04)
 		)
@@
 	(wire
 		(pts
-			(xy 209.55 66.04) (xy 227.33 66.04)
+			(xy 209.55 66.04) (xy 215.9 66.04)
 		)
 		(stroke
@@
 	(wire
 		(pts
-			(xy 163.83 86.36) (xy 179.07 86.36)
-		)
-		(stroke
-			(width 0)
-			(type default)
-		)
-	)
-	(wire
-		(pts
 			(xy 209.55 83.82) (xy 209.55 86.36)
 		)
@@
 	)
 	(symbol
-		(lib_id "Spartanpods_SymbolLibrary:Fiducial")
+		(lib_id "Spartanpods_v4_SymbolLibrary:Fiducial")
 		(at 267.97 140.97 0)
 		(unit 1)
@@
 	)
 	(symbol
-		(lib_id "Spartanpods_SymbolLibrary:PWR_FLAG")
+		(lib_id "Spartanpods_v4_SymbolLibrary:PWR_FLAG")
 		(at 76.2 81.28 90)
 		(unit 1)
@@
 	)
 	(symbol
-		(lib_id "Spartanpods_SymbolLibrary:LED")
+		(lib_id "Spartanpods_v4_SymbolLibrary:LED")
 		(at 267.97 80.01 90)
 		(unit 1)
@@
 	)
 	(symbol
-		(lib_id "Spartanpods_SymbolLibrary:LED")
+		(lib_id "Spartanpods_v4_SymbolLibrary:LED")
 		(at 199.39 80.01 90)
 		(unit 1)
@@
 	)
 	(symbol
-		(lib_id "Spartanpods_SymbolLibrary:R_US")
+		(lib_id "Spartanpods_v4_SymbolLibrary:R_US")
 		(at 199.39 71.12 0)
 		(unit 1)
@@
 	)
 	(symbol
-		(lib_id "Spartanpods_SymbolLibrary:R_US")
+		(lib_id "Spartanpods_v4_SymbolLibrary:R_US")
 		(at 156.21 71.12 0)
 		(unit 1)
@@
 	)
 	(symbol
-		(lib_id "Spartanpods_SymbolLibrary:+3.3V")
+		(lib_id "Spartanpods_v4_SymbolLibrary:+3.3V")
 		(at 76.2 66.04 0)
 		(unit 1)
@@
 	)
 	(symbol
-		(lib_id "Spartanpods_SymbolLibrary:R_US")
+		(lib_id "Spartanpods_v4_SymbolLibrary:R_US")
 		(at 257.81 71.12 0)
 		(unit 1)
@@
 	)
 	(symbol
-		(lib_id "Spartanpods_SymbolLibrary:LED")
+		(lib_id "Spartanpods_v4_SymbolLibrary:LED")
 		(at 189.23 80.01 90)
 		(unit 1)
@@
 	)
 	(symbol
-		(lib_id "Spartanpods_SymbolLibrary:Logo_Open_Hardware_Small")
+		(lib_id "Spartanpods_v4_SymbolLibrary:Logo_Open_Hardware_Small")
 		(at 226.06 157.48 0)
 		(unit 1)
@@
 			)
 		)
-		(property "Footprint" "Spartanpods:Combined"
+		(property "Footprint" "Spartanpods:Combined_LED Text"
 			(at 226.06 157.48 0)
 			(effects
@@
 	)
 	(symbol
-		(lib_id "Spartanpods_SymbolLibrary:SW_DP3T")
+		(lib_id "Spartanpods_v4_SymbolLibrary:SW_DP3T")
 		(at 92.71 121.92 0)
 		(unit 1)
@@
 			)
 		)
-		(property "Footprint" ""
+		(property "Footprint" "!MyFootprints:DP3T - JS203011SCQN"
 			(at 76.835 117.475 0)
 			(effects
@@
 	)
 	(symbol
-		(lib_id "Spartanpods_SymbolLibrary:LED")
+		(lib_id "Spartanpods_v4_SymbolLibrary:LED")
 		(at 227.33 80.01 90)
 		(unit 1)
@@
 	)
 	(symbol
-		(lib_id "Device:R_US")
-		(at 163.83 90.17 0)
+		(lib_id "Spartanpods_v4_SymbolLibrary:R_US")
+		(at 219.71 66.04 90)
 		(unit 1)
 		(exclude_from_sim no)
@@
 		(fields_autoplaced yes)
 		(property "Reference" "R12"
-			(at 166.37 88.8999 0)
+			(at 219.71 59.69 90)
 			(effects
 				(font
 					(size 1.27 1.27)
 				)
-				(justify left)
 			)
 		)
 		(property "Value" "0 Ohm jumper"
-			(at 166.37 91.4399 0)
+			(at 219.71 62.23 90)
 			(effects
 				(font
 					(size 1.27 1.27)
 				)
-				(justify left)
 			)
 		)
-		(property "Footprint" ""
-			(at 164.846 90.424 90)
+		(property "Footprint" "Resistor_SMD:R_0805_2012Metric_Pad1.20x1.40mm_HandSolder"
+			(at 219.964 65.024 90)
 			(effects
 				(font
@@
 		)
 		(property "Datasheet" "~"
-			(at 163.83 90.17 0)
+			(at 219.71 66.04 0)
 			(effects
 				(font
@@
 		)
 		(property "Description" "Resistor, US symbol"
-			(at 163.83 90.17 0)
+			(at 219.71 66.04 0)
 			(effects
 				(font
@@
 	)
 	(symbol
-		(lib_id "Spartanpods_SymbolLibrary:R_US")
+		(lib_id "Spartanpods_v4_SymbolLibrary:R_US")
 		(at 179.07 71.12 0)
 		(unit 1)
@@
 	)
 	(symbol
-		(lib_id "Spartanpods_SymbolLibrary:LED")
+		(lib_id "Spartanpods_v4_SymbolLibrary:LED")
 		(at 179.07 80.01 90)
 		(unit 1)
@@
 	)
 	(symbol
-		(lib_id "Spartanpods_SymbolLibrary:LED")
+		(lib_id "Spartanpods_v4_SymbolLibrary:LED")
 		(at 156.21 80.01 90)
 		(unit 1)
@@
 	)
 	(symbol
-		(lib_id "Spartanpods_SymbolLibrary:R_Potentiometer_US")
+		(lib_id "Spartanpods_v4_SymbolLibrary:R_Potentiometer_US")
 		(at 116.84 90.17 0)
 		(unit 1)
@@
 	)
 	(symbol
-		(lib_id "Spartanpods_SymbolLibrary:Fiducial")
+		(lib_id "Spartanpods_v4_SymbolLibrary:Fiducial")
 		(at 267.97 153.67 0)
 		(unit 1)
@@
 	)
 	(symbol
-		(lib_id "Spartanpods_SymbolLibrary:Fiducial")
+		(lib_id "Spartanpods_v4_SymbolLibrary:Fiducial")
 		(at 267.97 160.02 0)
 		(unit 1)
@@
 	)
 	(symbol
-		(lib_id "Spartanpods_SymbolLibrary:LED")
+		(lib_id "Spartanpods_v4_SymbolLibrary:LED")
 		(at 237.49 80.01 90)
 		(unit 1)
@@
 	)
 	(symbol
-		(lib_id "Spartanpods_SymbolLibrary:GNDREF")
+		(lib_id "Spartanpods_v4_SymbolLibrary:GNDREF")
 		(at 76.2 125.73 0)
 		(unit 1)
@@
 	)
 	(symbol
-		(lib_id "Spartanpods_SymbolLibrary:R_US")
+		(lib_id "Spartanpods_v4_SymbolLibrary:R_US")
 		(at 267.97 71.12 0)
 		(unit 1)
@@
 	)
 	(symbol
-		(lib_id "Spartanpods_SymbolLibrary:LED")
+		(lib_id "Spartanpods_v4_SymbolLibrary:LED")
 		(at 257.81 80.01 90)
 		(unit 1)
@@
 	)
 	(symbol
-		(lib_id "Spartanpods_SymbolLibrary:BC847")
+		(lib_id "Spartanpods_v4_SymbolLibrary:BC847")
 		(at 142.24 100.33 0)
 		(unit 1)
@@
 	)
 	(symbol
-		(lib_id "Spartanpods_SymbolLibrary:R_US")
+		(lib_id "Spartanpods_v4_SymbolLibrary:R_US")
 		(at 227.33 71.12 0)
 		(unit 1)
@@
 	)
 	(symbol
-		(lib_id "Spartanpods_SymbolLibrary:LED")
+		(lib_id "Spartanpods_v4_SymbolLibrary:LED")
 		(at 209.55 80.01 90)
 		(unit 1)
@@
 	)
 	(symbol
-		(lib_id "Spartanpods_SymbolLibrary:R_US")
+		(lib_id "Spartanpods_v4_SymbolLibrary:R_US")
 		(at 247.65 71.12 0)
 		(unit 1)
@@
 	)
 	(symbol
-		(lib_id "Spartanpods_SymbolLibrary:Fiducial")
+		(lib_id "Spartanpods_v4_SymbolLibrary:Fiducial")
 		(at 267.97 147.32 0)
 		(unit 1)
@@
 	)
 	(symbol
-		(lib_id "Spartanpods_SymbolLibrary:R_US")
+		(lib_id "Spartanpods_v4_SymbolLibrary:R_US")
 		(at 209.55 71.12 0)
 		(unit 1)
@@
 	)
 	(symbol
-		(lib_id "Spartanpods_SymbolLibrary:R_US")
+		(lib_id "Spartanpods_v4_SymbolLibrary:R_US")
 		(at 189.23 71.12 0)
 		(unit 1)
@@
 	)
 	(symbol
-		(lib_id "Spartanpods_SymbolLibrary:R_US")
+		(lib_id "Spartanpods_v4_SymbolLibrary:R_US")
 		(at 116.84 76.2 0)
 		(mirror x)
@@
 	)
 	(symbol
-		(lib_id "Spartanpods_SymbolLibrary:SW_DP3T")
+		(lib_id "Spartanpods_v4_SymbolLibrary:SW_DP3T")
 		(at 92.71 133.35 0)
 		(unit 2)
@@
 			)
 		)
-		(property "Footprint" ""
+		(property "Footprint" "!MyFootprints:DP3T - JS203011SCQN"
 			(at 76.835 128.905 0)
 			(effects
@@
 	)
 	(symbol
-		(lib_id "Spartanpods_SymbolLibrary:Battery_Cell")
+		(lib_id "Spartanpods_v4_SymbolLibrary:Battery_Cell")
 		(at 76.2 95.25 0)
 		(mirror y)
@@
 	)
 	(symbol
-		(lib_id "Spartanpods_SymbolLibrary:LED")
+		(lib_id "Spartanpods_v4_SymbolLibrary:LED")
 		(at 247.65 80.01 90)
 		(unit 1)
@@
 	)
 	(symbol
-		(lib_id "Spartanpods_SymbolLibrary:JD3_Diode")
+		(lib_id "Spartanpods_v4_SymbolLibrary:JD3_Diode")
 		(at 241.3 157.48 0)
 		(unit 1)
@@
 	)
 	(symbol
-		(lib_id "Spartanpods_SymbolLibrary:R_US")
+		(lib_id "Spartanpods_v4_SymbolLibrary:R_US")
 		(at 237.49 71.12 0)
 		(unit 1)
@@
 	)
 	(symbol
-		(lib_id "Spartanpods_SymbolLibrary:Q_Photo_NPN")
+		(lib_id "Spartanpods_v4_SymbolLibrary:Q_Photo_NPN")
 		(at 121.92 107.95 0)
 		(unit 1)
@@
 	)
 	(symbol
-		(lib_id "Spartanpods_SymbolLibrary:PWR_FLAG")
+		(lib_id "Spartanpods_v4_SymbolLibrary:PWR_FLAG")
 		(at 76.2 106.68 90)
 		(unit 1)
